File: synth_vco.sch (KiCad schematic (older format))
At the start: 22 parts, among them J1 PWR, SW1 SW_SPDT, U1 TL081

Commit message: 2
Parts:
- SW1: footprint (none) -> Button_Switch_THT:SW_E-Switch_EG1271_DPDT
- U1: footprint Package_SO:SOP-8_3.9x4.9mm_P1.27mm -> Package_SO:SOIC-8_3.9x4.9mm_P1.27mm
Changed lines of the file:
@@
 F 0 "U1" H 4200 3600 50  0000 L CNN
 F 1 "TL081" H 4200 3350 50  0000 L CNN
-F 2 "Package_SO:SOP-8_3.9x4.9mm_P1.27mm" H 4100 3550 50  0001 C CNN
+F 2 "Package_SO:SOIC-8_3.9x4.9mm_P1.27mm" H 4100 3550 50  0001 C CNN
 F 3 "http://www.ti.com/lit/ds/symlink/tl081.pdf" H 4200 3650 50  0001 C CNN
 	1    4050 3500
@@
 F 0 "SW1" H 2800 4135 50  0000 C CNN
 F 1 "SW_SPDT" H 2800 4044 50  0000 C CNN
-F 2 "" H 2800 3850 50  0001 C CNN
+F 2 "Button_Switch_THT:SW_E-Switch_EG1271_DPDT" H 2800 3850 50  0001 C CNN
 F 3 "~" H 2800 3850 50  0001 C CNN
 	1    2800 3850
