File: synth_vco.kicad_pcb (KiCad board)
At the start: 2 copper layers, 160 x 50 mm, 21 parts, among them J1 PWR, U1 TL081

Commit message: 2
Parts:
- added SW1: SW_SPDT, Button_Switch_THT:SW_E-Switch_EG1271_DPDT, F.Cu at (83.1, 82.5)
- U1: footprint Package_SO:SOP-8_3.9x4.9mm_P1.27mm -> Package_SO:SOIC-8_3.9x4.9mm_P1.27mm
- moved R1 45.6 mm to (105.2, 61.2), turned to 90 degrees
- moved R5 41.8 mm to (119.9, 61.8)
- moved R9 41.8 mm to (119.9, 58.7)
- moved RV1 41.3 mm to (95.2, 67.6)
- moved RV3 41.3 mm to (95.2, 60.0)
- moved RV5 41.3 mm to (95.2, 52.4)
- moved U1 41.3 mm to (111.8, 57.2)
- moved R4 41.3 mm to (89.2, 60.0)
- moved R6 41.3 mm to (89.2, 55.2)
- moved RV4 41.1 mm to (120.7, 52.9)
- moved R7 40.6 mm to (101.9, 61.2), turned to 90 degrees
- moved R10 40.3 mm to (101.9, 56.9), turned to 90 degrees
- moved R2 33.5 mm to (108.2, 66.4), turned to 90 degrees
- moved R3 33.3 mm to (105.2, 66.4), turned to 90 degrees
- moved R8 25.9 mm to (105.2, 56.9), turned to 270 degrees
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Connections:
- R2 pad 1: (no net) -> Net-(R2-Pad1)
Routing:
- net -15V: track 45.5 -> 0.00 mm, vias 1 -> 0
- net +15V: track 37.8 -> 0.00 mm, vias 1 -> 0
- net /DC_OFFSET: track 19.8 -> 0.00 mm
- net Net-(R3-Pad1): track 13.5 -> 0.00 mm
- net Net-(R4-Pad2): track 7.95 -> 0.00 mm
- net Net-(R7-Pad1): track 4.20 -> 0.00 mm
- net Net-(R10-Pad2): track 4.20 -> 0.00 mm
- net Net-(R1-Pad1): track 4.20 -> 0.00 mm
- removed copper zone on F.Cu, net GND
Other:
- board outline removed

Commit message: message
Parts:
- moved R7 40.4 mm to (61.7, 66.0), turned to 0 degrees
- moved RV3 39.1 mm to (56.1, 60.7), turned to 90 degrees
- moved R3 38.5 mm to (67.3, 73.7), turned to 0 degrees
- moved R1 38.3 mm to (67.3, 67.0)
- moved R8 37.1 mm to (72.0, 73.7), turned to 180 degrees
- moved RV1 36.1 mm to (59.4, 71.9)
- moved R5 34.0 mm to (88.4, 74.7)
- moved R9 33.8 mm to (88.4, 71.1), turned to 0 degrees
- moved U1 33.1 mm to (80.3, 67.3)
- moved R10 32.3 mm to (71.1, 67.0)
- moved RV4 30.9 mm to (91.7, 63.6), turned to 180 degrees
- moved R2 30.8 mm to (79.6, 77.9)
- moved R4 30.3 mm to (59.4, 54.6), turned to 180 degrees
- moved RV5 29.2 mm to (67.3, 60.7), turned to 90 degrees
- moved R6 25.0 mm to (64.1, 54.6), turned to 0 degrees
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